File: PCB/NyxNodsMotherboard/NyxNodsMotherboard.kicad_pcb (KiCad board)
At the start: 4 copper layers, 190.8 x 101 mm, 51 parts, among them J1 2130830005, J2 CPG-04-TH-TR, J3 S2B-PH-SM4-TB_LF__SN_, J4 2065-100/998-403, J5 2130830005, J6 2065-100/998-403, J7 CPG-04-TH-TR, U1 BQ24072TRGTR, U2 TPS62842DGRR

Commit message: Layout Progress, 3D models imported
Parts:
- moved R20 101.9 mm to (210.5, 101.7), turned to -90 degrees
- moved C7 98.2 mm to (170.2, 140.8), turned to 90 degrees
- moved R19 96.7 mm to (203.8, 102.5), turned to 180 degrees
- moved R4 95.0 mm to (175.2, 134.2)
- moved R3 94.6 mm to (175.2, 131.8), turned to 180 degrees
- moved R14 91.9 mm to (164.8, 138.2)
- moved C6 90.9 mm to (156.8, 140.2), turned to -90 degrees
- moved R15 89.2 mm to (164.8, 137.2)
- moved U2 87.2 mm to (160.5, 140.0), turned to 180 degrees
- moved R18 86.9 mm to (156.8, 138.2), turned to 90 degrees
- moved R6 86.6 mm to (156.8, 134.2), turned to 180 degrees
- moved L1 80.2 mm to (166.8, 141.2)
- moved R5 79.1 mm to (156.8, 131.2), turned to 180 degrees
- moved D2 73.6 mm to (175.8, 135.7), turned to -90 degrees
- moved D4 72.8 mm to (228.2, 138.5)
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Other:
- board size 190.8 x 101 mm -> 31.1 x 26.8 mm
